File: KiCad/taro.kicad_pcb (KiCad board)
At the start: 2 copper layers, 115.6 x 77.5 mm, 35 parts, among them J1 Conn_01x04_Female, SW1 Reset, SW10 SW_Push, SW11 SW_Push, SW12 SW_Push, SW13 SW_Push, SW14 Rotary_Encoder_Switch, SW15 SW_Push, SW16 SW_Push, SW17 SW_Push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

Commit message: Added mounting holes
Parts:
- added HOLE5: MountingHole_4mm, Keyboard_Parts:MountingHole_M2, F.Cu at (139.7, 73.0)
- added HOLE5: MountingHole_4mm, Keyboard_Parts:MountingHole_M2, F.Cu at (139.7, 130.2)
- added HOLE5: MountingHole_4mm, Keyboard_Parts:MountingHole_M2, F.Cu at (63.5, 130.2)
- added HOLE5: MountingHole_4mm, Keyboard_Parts:MountingHole_M2, F.Cu at (63.5, 73.0)
Changed lines of the file:
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@@
     (tracks 0)
     (zones 0)
-    (modules 35)
+    (modules 39)
     (nets 34)
   )
@@
     (solder_mask_min_width 0.25)
     (aux_axis_origin 0 0)
-    (visible_elements FFFFF77F)
+    (visible_elements 7FFFF7FF)
     (pcbplotparams
       (layerselection 0x010f0_ffffffff)
@@
     (add_net VCC)
   )
+  (module Keyboard_Parts:MountingHole_M2 (layer F.Cu)
+    (at 139.7 73.025)
+    (descr "Mounting Hole 4mm, no annular")
+    (tags "mounting hole 4mm no annular")
+    (attr virtual)
+    (fp_text reference HOLE5 (at 0 -5) (layer F.SilkS) hide
+      (effects (font (size 1 1) (thickness 0.15)))
+    )
+    (fp_text value MountingHole_4mm (at 0 5) (layer F.Fab)
+      (effects (font (size 1 1) (thickness 0.15)))
+    )
+    (fp_text user %R (at -5.5 0 90) (layer F.Fab)
+      (effects (font (size 1 1) (thickness 0.15)))
+    )
+    (fp_circle (center 0 0) (end 3 0) (layer Cmts.User) (width 0.15))
+    (fp_circle (center 0 0) (end 4.25 0) (layer F.CrtYd) (width 0.05))
+    (pad 1 thru_hole circle (at 0 0) (size 3.3 3.3) (drill 2.3) (layers *.Cu *.Mask))
+  )
+  (module Keyboard_Parts:MountingHole_M2 (layer F.Cu)
+    (at 139.7 130.175)
+    (descr "Mounting Hole 4mm, no annular")
+    (tags "mounting hole 4mm no annular")
+    (attr virtual)
+    (fp_text reference HOLE5 (at 0 -5) (layer F.SilkS) hide
+      (effects (font (size 1 1) (thickness 0.15)))
+    )
+    (fp_text value MountingHole_4mm (at 0 5) (layer F.Fab)
+      (effects (font (size 1 1) (thickness 0.15)))
+    )
+    (fp_text user %R (at -5.5 0 90) (layer F.Fab)
+      (effects (font (size 1 1) (thickness 0.15)))
+    )
+    (fp_circle (center 0 0) (end 3 0) (layer Cmts.User) (width 0.15))
+    (fp_circle (center 0 0) (end 4.25 0) (layer F.CrtYd) (width 0.05))
+    (pad 1 thru_hole circle (at 0 0) (size 3.3 3.3) (drill 2.3) (layers *.Cu *.Mask))
+  )
+  (module Keyboard_Parts:MountingHole_M2 (layer F.Cu)
+    (at 63.5 130.175)
+    (descr "Mounting Hole 4mm, no annular")
+    (tags "mounting hole 4mm no annular")
+    (attr virtual)
+    (fp_text reference HOLE5 (at 0 -5) (layer F.SilkS) hide
+      (effects (font (size 1 1) (thickness 0.15)))
+    )
+    (fp_text value MountingHole_4mm (at 0 5) (layer F.Fab)
+      (effects (font (size 1 1) (thickness 0.15)))
+    )
+    (fp_text user %R (at -5.5 0 90) (layer F.Fab)
+      (effects (font (size 1 1) (thickness 0.15)))
+    )
+    (fp_circle (center 0 0) (end 3 0) (layer Cmts.User) (width 0.15))
+    (fp_circle (center 0 0) (end 4.25 0) (layer F.CrtYd) (width 0.05))
+    (pad 1 thru_hole circle (at 0 0) (size 3.3 3.3) (drill 2.3) (layers *.Cu *.Mask))
+  )
+  (module Keyboard_Parts:MountingHole_M2 (layer F.Cu)
+    (at 63.5 73.025)
+    (descr "Mounting Hole 4mm, no annular")
+    (tags "mounting hole 4mm no annular")
+    (attr virtual)
+    (fp_text reference HOLE5 (at 0 -5) (layer F.SilkS) hide
+      (effects (font (size 1 1) (thickness 0.15)))
+    )
+    (fp_text value MountingHole_4mm (at 0 5) (layer F.Fab)
+      (effects (font (size 1 1) (thickness 0.15)))
+    )
+    (fp_text user %R (at -5.5 0 90) (layer F.Fab)
+      (effects (font (size 1 1) (thickness 0.15)))
+    )
+    (fp_circle (center 0 0) (end 3 0) (layer Cmts.User) (width 0.15))
+    (fp_circle (center 0 0) (end 4.25 0) (layer F.CrtYd) (width 0.05))
+    (pad 1 thru_hole circle (at 0 0) (size 3.3 3.3) (drill 2.3) (layers *.Cu *.Mask))
+  )
   (module Keebio_Parts:ArduinoProMicro (layer F.Cu)
