File: pcb/taro.kicad_pcb (KiCad board)
At the start: 2 copper layers, 115.6 x 77.5 mm, 39 parts, among them J1 Conn_01x04_Female, SW1 Reset, SW10 SW_Push, SW11 SW_Push, SW12 SW_Push, SW13 SW_Push, SW14 Rotary_Encoder_Switch, SW15 SW_Push, SW16 SW_Push, SW17 SW_Push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

Commit message: pcb ready for art
Parts:
- removed HOLE5 (x4): MountingHole_4mm, Keyboard_Parts:MountingHole_M2
- SW10, SW11, SW12, SW13, SW15, SW16, SW17, SW2, SW3, SW4, SW5, SW6, SW7, SW8, SW9: footprint TheKeebrary:MX_PCB_100H -> TheKeebrary:Hybrid_PCB_100H
- moved SW1 47.6 mm to (127.0, 66.0)
Routing:
- net /ROW_D: track 0.00 -> 148.3 mm
- net /ROW_C: track 0.00 -> 125.1 mm, vias 0 -> 4
- net /COL_A: track 0.00 -> 111.7 mm
- net /COL_B: track 0.00 -> 94.7 mm
- net /COL_F: track 0.00 -> 81.1 mm, vias 0 -> 1
- net /COL_C: track 0.00 -> 80.4 mm
- net /COL_D: track 0.00 -> 79.5 mm
- net /COL_E: track 0.00 -> 60.1 mm, vias 0 -> 1
- net /ROW_B: track 0.00 -> 56.8 mm, vias 0 -> 4
- net /ROT1_B: track 0.00 -> 47.5 mm
- net VCC: track 0.00 -> 42.8 mm
- net /ROT1_A: track 0.00 -> 41.6 mm
- net /ROW_A: track 0.00 -> 40.7 mm, vias 0 -> 2
- net Net-(SW1-Pad1): track 0.00 -> 39.0 mm
- net /SDA: track 0.00 -> 19.6 mm
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- added copper zone on B.Cu, net GND
- added copper zone on F.Cu, net GND
