File: pcb/taro.kicad_pcb (KiCad board)
At the start: 2 copper layers, 115.6 x 77.5 mm, 35 parts, among them J1 Conn_01x04_Female, SW1 Reset, SW10 SW_Push, SW11 SW_Push, SW12 SW_Push, SW13 SW_Push, SW14 Rotary_Encoder_Switch, SW15 SW_Push, SW16 SW_Push, SW17 SW_Push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

Commit message: en tiiä
Parts:
- added G***: LOGO, art:top_art, F.Cu at (101.0, 101.6)
