File: pcb/taro.kicad_pcb (KiCad board)
At the start: 2 copper layers, 115.6 x 77.5 mm, 37 parts, among them J1 Conn_01x04_Female, SW1 Reset, SW10 SW_Push, SW11 SW_Push, SW12 SW_Push, SW13 SW_Push, SW14 PEC16-S, SW15 SW_Push, SW16 SW_Push, SW17 SW_Push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

Commit message: pcb done
Parts:
- added D17: WS2812B, LEDs:LED_WS2812B-PLCC4, B.Cu at (139.7, 66.0)
- added D18: WS2812B, LEDs:LED_WS2812B-PLCC4, B.Cu at (139.7, 101.6)
- added D19: WS2812B, LEDs:LED_WS2812B-PLCC4, B.Cu at (139.7, 137.2)
- added D20: WS2812B, LEDs:LED_WS2812B-PLCC4, B.Cu at (101.6, 137.2)
- added D21: WS2812B, LEDs:LED_WS2812B-PLCC4, B.Cu at (63.5, 137.2)
- added D22: WS2812B, LEDs:LED_WS2812B-PLCC4, B.Cu at (63.5, 101.6)
- added D23: WS2812B, LEDs:LED_WS2812B-PLCC4, B.Cu at (63.5, 66.0)
- added H1: MountingHole, Keyboard_Parts:MountingHole_M2, F.Cu at (63.5, 73.0)
- added H2: MountingHole, Keyboard_Parts:MountingHole_M2, F.Cu at (63.5, 130.2)
- added H3: MountingHole, Keyboard_Parts:MountingHole_M2, F.Cu at (139.7, 73.0)
- added H4: MountingHole, Keyboard_Parts:MountingHole_M2, F.Cu at (139.7, 130.2)
- SW14: value PEC16-S -> SW_Push; footprint Avp:PEC16-4xxxF-Sxxxx -> TheKeebrary:Hybrid_PCB_100H
- SW17: value SW_Push -> Rotary_Encoder_Switch; footprint TheKeebrary:Hybrid_PCB_100H -> Keebio_Parts:RotaryEncoder_Alps_EC11E-Switch_Vertical_H20mm
- moved SW14 42.6 mm to (111.1, 130.2)
- moved SW17 42.6 mm to (130.2, 92.1), turned to 90 degrees
- moved SW15 19.1 mm to (130.2, 130.2)
- moved SW16 19.0 mm to (149.2, 130.2)
- moved G*** 2.62 mm to (129.5, 109.9)
- moved G*** 1.27 mm to (101.6, 101.6)
- turned D14 to 180 degrees
Connections:
- SW14 pad 1: /ROT1_A -> /COL_D
- SW14 pad 2: /ROT1_B -> Net-(D13-Pad2)
- SW15 pad 1: /COL_D -> /COL_E
- SW15 pad 2: Net-(D13-Pad2) -> Net-(D15-Pad2)
- SW16 pad 1: /COL_E -> /COL_F
- SW16 pad 2: Net-(D15-Pad2) -> Net-(D16-Pad2)
- U1 pad 19: (no net) -> /LED_IN
Routing:
- net VCC: track 42.8 -> 286.8 mm, vias 0 -> 7
- net Net-(D20-Pad2): track 0.00 -> 46.5 mm, vias 0 -> 4
- net Net-(D21-Pad2): track 0.00 -> 46.1 mm, vias 0 -> 2
- net Net-(D19-Pad2): track 0.00 -> 44.6 mm, vias 0 -> 2
- net /LED_IN: track 0.00 -> 44.5 mm
- net Net-(D22-Pad2): track 0.00 -> 44.0 mm, vias 0 -> 2
- net Net-(D17-Pad2): track 0.00 -> 35.0 mm
- net Net-(D18-Pad2): track 0.00 -> 34.4 mm
- net /COL_F: track 81.2 -> 62.4 mm, vias 1 -> 0
- net /COL_E: track 60.2 -> 47.9 mm, vias 1 -> 0
- net /ROW_C: track 117.5 -> 126.1 mm
- net /ROT1_B: track 46.2 -> 40.0 mm
- net /ROT1_A: track 40.2 -> 34.0 mm
- net /COL_A: track 111.7 -> 114.4 mm
- net /ROW_A: track 40.7 -> 42.7 mm
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