File: pcb/taro.sch (KiCad schematic (older format))
At the start: 35 parts, among them J1 Conn_01x04_Female, SW1 Reset, SW10 SW_Push, SW11 SW_Push, SW12 SW_Push, SW13 SW_Push, SW14 Rotary_Encoder_Switch, SW15 SW_Push, SW16 SW_Push, SW17 SW_Push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

Commit message: pcb ready for art
Parts:
- SW10, SW11, SW12, SW13, SW15, SW16, SW17, SW2, SW3, SW4, SW5, SW6, SW7, SW8, SW9: footprint TheKeebrary:MX_PCB_100H -> TheKeebrary:Hybrid_PCB_100H
Changed lines of the file:
@@
 F 0 "SW2" H 4400 2585 50  0000 C CNN
 F 1 "SW_Push" H 4400 2494 50  0000 C CNN
-F 2 "TheKeebrary:MX_PCB_100H" H 4400 2500 50  0001 C CNN
+F 2 "TheKeebrary:Hybrid_PCB_100H" H 4400 2500 50  0001 C CNN
 F 3 "~" H 4400 2500 50  0001 C CNN
 	1    4400 2300
@@
 F 0 "SW3" H 4400 3235 50  0000 C CNN
 F 1 "SW_Push" H 4400 3144 50  0000 C CNN
-F 2 "TheKeebrary:MX_PCB_100H" H 4400 3150 50  0001 C CNN
+F 2 "TheKeebrary:Hybrid_PCB_100H" H 4400 3150 50  0001 C CNN
 F 3 "~" H 4400 3150 50  0001 C CNN
 	1    4400 2950
@@
 F 0 "SW4" H 4400 3885 50  0000 C CNN
 F 1 "SW_Push" H 4400 3794 50  0000 C CNN
-F 2 "TheKeebrary:MX_PCB_100H" H 4400 3800 50  0001 C CNN
+F 2 "TheKeebrary:Hybrid_PCB_100H" H 4400 3800 50  0001 C CNN
 F 3 "~" H 4400 3800 50  0001 C CNN
 	1    4400 3600
@@
 F 0 "SW5" H 4400 4535 50  0000 C CNN
 F 1 "SW_Push" H 4400 4444 50  0000 C CNN
-F 2 "TheKeebrary:MX_PCB_100H" H 4400 4450 50  0001 C CNN
+F 2 "TheKeebrary:Hybrid_PCB_100H" H 4400 4450 50  0001 C CNN
 F 3 "~" H 4400 4450 50  0001 C CNN
 	1    4400 4250
@@
 F 0 "SW6" H 5050 2585 50  0000 C CNN
 F 1 "SW_Push" H 5050 2494 50  0000 C CNN
-F 2 "TheKeebrary:MX_PCB_100H" H 5050 2500 50  0001 C CNN
+F 2 "TheKeebrary:Hybrid_PCB_100H" H 5050 2500 50  0001 C CNN
 F 3 "~" H 5050 2500 50  0001 C CNN
 	1    5050 2300
@@
 F 0 "SW7" H 5050 3235 50  0000 C CNN
 F 1 "SW_Push" H 5050 3144 50  0000 C CNN
-F 2 "TheKeebrary:MX_PCB_100H" H 5050 3150 50  0001 C CNN
+F 2 "TheKeebrary:Hybrid_PCB_100H" H 5050 3150 50  0001 C CNN
 F 3 "~" H 5050 3150 50  0001 C CNN
 	1    5050 2950
@@
 F 0 "SW8" H 5050 3885 50  0000 C CNN
 F 1 "SW_Push" H 5050 3794 50  0000 C CNN
-F 2 "TheKeebrary:MX_PCB_100H" H 5050 3800 50  0001 C CNN
+F 2 "TheKeebrary:Hybrid_PCB_100H" H 5050 3800 50  0001 C CNN
 F 3 "~" H 5050 3800 50  0001 C CNN
 	1    5050 3600
@@
 F 0 "SW9" H 5050 4535 50  0000 C CNN
 F 1 "SW_Push" H 5050 4444 50  0000 C CNN
-F 2 "TheKeebrary:MX_PCB_100H" H 5050 4450 50  0001 C CNN
+F 2 "TheKeebrary:Hybrid_PCB_100H" H 5050 4450 50  0001 C CNN
 F 3 "~" H 5050 4450 50  0001 C CNN
 	1    5050 4250
@@
 F 0 "SW13" H 5700 4535 50  0000 C CNN
 F 1 "SW_Push" H 5700 4444 50  0000 C CNN
-F 2 "TheKeebrary:MX_PCB_100H" H 5700 4450 50  0001 C CNN
+F 2 "TheKeebrary:Hybrid_PCB_100H" H 5700 4450 50  0001 C CNN
 F 3 "~" H 5700 4450 50  0001 C CNN
 	1    5700 4250
@@
 F 0 "SW12" H 5700 3885 50  0000 C CNN
 F 1 "SW_Push" H 5700 3794 50  0000 C CNN
-F 2 "TheKeebrary:MX_PCB_100H" H 5700 3800 50  0001 C CNN
+F 2 "TheKeebrary:Hybrid_PCB_100H" H 5700 3800 50  0001 C CNN
 F 3 "~" H 5700 3800 50  0001 C CNN
 	1    5700 3600
@@
 F 0 "SW11" H 5700 3235 50  0000 C CNN
 F 1 "SW_Push" H 5700 3144 50  0000 C CNN
-F 2 "TheKeebrary:MX_PCB_100H" H 5700 3150 50  0001 C CNN
+F 2 "TheKeebrary:Hybrid_PCB_100H" H 5700 3150 50  0001 C CNN
 F 3 "~" H 5700 3150 50  0001 C CNN
 	1    5700 2950
@@
 F 0 "SW10" H 5700 2585 50  0000 C CNN
 F 1 "SW_Push" H 5700 2494 50  0000 C CNN
-F 2 "TheKeebrary:MX_PCB_100H" H 5700 2500 50  0001 C CNN
+F 2 "TheKeebrary:Hybrid_PCB_100H" H 5700 2500 50  0001 C CNN
 F 3 "~" H 5700 2500 50  0001 C CNN
 	1    5700 2300
@@
 F 0 "SW17" H 7850 4535 50  0000 C CNN
 F 1 "SW_Push" H 7850 4444 50  0000 C CNN
-F 2 "TheKeebrary:MX_PCB_100H" H 7850 4450 50  0001 C CNN
+F 2 "TheKeebrary:Hybrid_PCB_100H" H 7850 4450 50  0001 C CNN
 F 3 "~" H 7850 4450 50  0001 C CNN
 	1    7850 4250
@@
 F 0 "SW16" H 7200 4535 50  0000 C CNN
 F 1 "SW_Push" H 7200 4444 50  0000 C CNN
-F 2 "TheKeebrary:MX_PCB_100H" H 7200 4450 50  0001 C CNN
+F 2 "TheKeebrary:Hybrid_PCB_100H" H 7200 4450 50  0001 C CNN
 F 3 "~" H 7200 4450 50  0001 C CNN
 	1    7200 4250
@@
 F 0 "SW15" H 6550 4535 50  0000 C CNN
 F 1 "SW_Push" H 6550 4444 50  0000 C CNN
-F 2 "TheKeebrary:MX_PCB_100H" H 6550 4450 50  0001 C CNN
+F 2 "TheKeebrary:Hybrid_PCB_100H" H 6550 4450 50  0001 C CNN
 F 3 "~" H 6550 4450 50  0001 C CNN
 	1    6550 4250

Commit message: pcb done?
Parts:
- removed SW14: Rotary_Encoder_Switch, Keebio_Parts:RotaryEncoder_Alps_EC11E-Switch_Vertical_H20mm, symbol Device:Rotary_Encoder_Switch
- added SW14: PEC16-S, Avp:PEC16-4xxxF-Sxxxx, symbol avp:PEC16-S
- U1: footprint Keebio_Parts:ArduinoProMicro -> Keebio_Parts:ArduinoProMicro-TopSide
Other:
- moved on the sheet: D14
Changed lines of the file:
@@
 F 0 "U1" H 2100 4687 60  0000 C CNN
 F 1 "ProMicro" H 2100 4581 60  0000 C CNN
-F 2 "Keebio_Parts:ArduinoProMicro" H 2200 2600 60  0001 C CNN
+F 2 "Keebio_Parts:ArduinoProMicro-TopSide" H 2200 2600 60  0001 C CNN
 F 3 "" H 2200 2600 60  0000 C CNN
 	1    2100 3650
@@
 	0    1    1    0
 $EndComp
-$Comp
-L Device:Rotary_Encoder_Switch SW14
-U 1 1 5F5EEC46
-P 6550 3250
-F 0 "SW14" H 6550 3617 50  0000 C CNN
-F 1 "Rotary_Encoder_Switch" H 6550 3526 50  0000 C CNN
-F 2 "Keebio_Parts:RotaryEncoder_Alps_EC11E-Switch_Vertical_H20mm" H 6400 3410 50  0001 C CNN
-F 3 "~" H 6550 3510 50  0001 C CNN
-	1    6550 3250
-	0    -1   -1   0
-$EndComp
 Wire Wire Line
 	5900 4550 6750 4550
 Connection ~ 5900 4550
 Wire Wire Line
-	5900 3900 6800 3900
+	5900 3900 6850 3900
 Connection ~ 5900 3900
 Connection ~ 5900 2600
@@
 L Device:D D14
 U 1 1 5F601314
-P 6800 3750
-F 0 "D14" V 6846 3671 50  0000 R CNN
-F 1 "D" V 6755 3671 50  0000 R CNN
-F 2 "Keebio_Parts:Diode" H 6800 3750 50  0001 C CNN
-F 3 "~" H 6800 3750 50  0001 C CNN
-	1    6800 3750
-	0    -1   -1   0
-$EndComp
-Wire Wire Line
-	6450 2950 6350 2950
-Connection ~ 6350 2950
-Wire Wire Line
-	6350 2950 6350 4250
-Wire Wire Line
-	6650 2950 6800 2950
-Wire Wire Line
-	6800 2950 6800 3600
-Text HLabel 6650 3550 3    50   Input ~ 0
+P 6850 3750
+F 0 "D14" V 6896 3671 50  0000 R CNN
+F 1 "D" V 6805 3671 50  0000 R CNN
+F 2 "Keebio_Parts:Diode" H 6850 3750 50  0001 C CNN
+F 3 "~" H 6850 3750 50  0001 C CNN
+	1    6850 3750
+	0    -1   -1   0
+$EndComp
+Text HLabel 6550 3300 3    50   Input ~ 0
 ROT1_B
-Text HLabel 6450 3550 3    50   Input ~ 0
-ROT1_A
 $Comp
 L power:GND #PWR08
 U 1 1 5F607E28
-P 6550 3550
-F 0 "#PWR08" H 6550 3300 50  0001 C CNN
-F 1 "GND" H 6555 3377 50  0000 C CNN
-F 2 "" H 6550 3550 50  0001 C CNN
-F 3 "" H 6550 3550 50  0001 C CNN
-	1    6550 3550
+P 6650 3300
+F 0 "#PWR08" H 6650 3050 50  0001 C CNN
+F 1 "GND" H 6655 3127 50  0000 C CNN
+F 2 "" H 6650 3300 50  0001 C CNN
+F 3 "" H 6650 3300 50  0001 C CNN
+	1    6650 3300
 	1    0    0    -1
 $EndComp
@@
 SDA
 Wire Wire Line
-	6350 1900 6350 2950
-Wire Wire Line
 	5900 2600 8050 2600
 Wire Wire Line
@@
 Wire Wire Line
 	7000 1900 7000 4250
+$Comp
+L avp:PEC16-S SW14
+U 1 1 5F5DF600
+P 6500 3000
+F 0 "SW14" V 7137 2692 60  0000 C CNN
+F 1 "PEC16-S" V 7031 2692 60  0000 C CNN
+F 2 "Avp:PEC16-4xxxF-Sxxxx" H 6500 3000 60  0001 C CNN
+F 3 "" H 6500 3000 60  0000 C CNN
+	1    6500 3000
+	0    -1   -1   0
+$EndComp
+Wire Wire Line
+	6350 1900 6350 3650
+Wire Wire Line
+	6850 3600 6850 3300
+Text HLabel 6450 3300 3    50   Input ~ 0
+ROT1_A
+Wire Wire Line
+	6750 3300 6750 3650
+Wire Wire Line
+	6750 3650 6350 3650
+Connection ~ 6350 3650
+Wire Wire Line
+	6350 3650 6350 4250
 $EndSCHEMATC

Commit message: pcb done
Parts:
- removed SW14: PEC16-S, Avp:PEC16-4xxxF-Sxxxx, symbol avp:PEC16-S
- added D17, D18, D19, D20, D21, D22, D23: WS2812B, LEDs:LED_WS2812B-PLCC4, symbol LED:WS2812B
- added H1, H2, H3, H4: MountingHole, Keyboard_Parts:MountingHole_M2, symbol Mechanical:MountingHole
- added SW17: Rotary_Encoder_Switch, Keebio_Parts:RotaryEncoder_Alps_EC11E-Switch_Vertical_H20mm, symbol Device:Rotary_Encoder_Switch
- renumbered SW15 to SW14, SW16 to SW15, SW17 to SW16
Connections:
- net labels added: LED_IN
Other:
- moved on the sheet: D14

Commit message: remove personal bom
Parts:
- U1: symbol Keebio:ProMicro -> taro-rescue:ProMicro-Keebio
Other:
- moved on the sheet: H1, H2, H3, H4, J1
Changed lines of the file:
@@
 $EndDescr
 $Comp
-L Keebio:ProMicro U1
+L taro-rescue:ProMicro-Keebio U1
 U 1 1 5F5954A3
 P 2100 3650
@@
 L Connector:Conn_01x04_Female J1
 U 1 1 5F60B0A1
-P 2050 1900
-F 0 "J1" V 1988 1612 50  0000 R CNN
-F 1 "Conn_01x04_Female" V 1897 1612 50  0000 R CNN
-F 2 "Pin_Headers:Pin_Header_Straight_1x04_Pitch2.54mm" H 2050 1900 50  0001 C CNN
-F 3 "~" H 2050 1900 50  0001 C CNN
-	1    2050 1900
+P 1550 7000
+F 0 "J1" V 1488 6712 50  0000 R CNN
+F 1 "Conn_01x04_Female" V 1397 6712 50  0000 R CNN
+F 2 "Pin_Headers:Pin_Header_Straight_1x04_Pitch2.54mm" H 1550 7000 50  0001 C CNN
+F 3 "~" H 1550 7000 50  0001 C CNN
+	1    1550 7000
 	0    -1   -1   0
 $EndComp
@@
 L power:GND #PWR04
 U 1 1 5F60E0F5
-P 2250 2100
-F 0 "#PWR04" H 2250 1850 50  0001 C CNN
-F 1 "GND" H 2255 1927 50  0000 C CNN
-F 2 "" H 2250 2100 50  0001 C CNN
-F 3 "" H 2250 2100 50  0001 C CNN
-	1    2250 2100
+P 1750 7200
+F 0 "#PWR04" H 1750 6950 50  0001 C CNN
+F 1 "GND" H 1755 7027 50  0000 C CNN
+F 2 "" H 1750 7200 50  0001 C CNN
+F 3 "" H 1750 7200 50  0001 C CNN
+	1    1750 7200
 	1    0    0    -1
 $EndComp
@@
 L power:VCC #PWR03
 U 1 1 5F60EBB5
-P 1950 2100
-F 0 "#PWR03" H 1950 1950 50  0001 C CNN
-F 1 "VCC" H 1968 2273 50  0000 C CNN
-F 2 "" H 1950 2100 50  0001 C CNN
-F 3 "" H 1950 2100 50  0001 C CNN
-	1    1950 2100
+P 1450 7200
+F 0 "#PWR03" H 1450 7050 50  0001 C CNN
+F 1 "VCC" H 1468 7373 50  0000 C CNN
+F 2 "" H 1450 7200 50  0001 C CNN
+F 3 "" H 1450 7200 50  0001 C CNN
+	1    1450 7200
 	-1   0    0    1
 $EndComp
-Text HLabel 2050 2100 3    50   Input ~ 0
+Text HLabel 1550 7200 3    50   Input ~ 0
 SCL
-Text HLabel 2150 2100 3    50   Input ~ 0
+Text HLabel 1650 7200 3    50   Input ~ 0
 SDA
 Wire Wire Line
@@
 L Mechanical:MountingHole H1
 U 1 1 5F62EDEA
-P 1700 4300
-F 0 "H1" H 1800 4346 50  0000 L CNN
-F 1 "MountingHole" H 1800 4255 50  0000 L CNN
-F 2 "Keyboard_Parts:MountingHole_M2" H 1700 4300 50  0001 C CNN
-F 3 "~" H 1700 4300 50  0001 C CNN
-	1    1700 4300
+P 1100 5750
+F 0 "H1" H 1200 5796 50  0000 L CNN
+F 1 "MountingHole" H 1200 5705 50  0000 L CNN
+F 2 "Keyboard_Parts:MountingHole_M2" H 1100 5750 50  0001 C CNN
+F 3 "~" H 1100 5750 50  0001 C CNN
+	1    1100 5750
 	1    0    0    -1
 $EndComp
@@
 L Mechanical:MountingHole H4
 U 1 1 5F6304BC
-P 1700 4900
-F 0 "H4" H 1800 4946 50  0000 L CNN
-F 1 "MountingHole" H 1800 4855 50  0000 L CNN
-F 2 "Keyboard_Parts:MountingHole_M2" H 1700 4900 50  0001 C CNN
-F 3 "~" H 1700 4900 50  0001 C CNN
-	1    1700 4900
+P 1100 6350
+F 0 "H4" H 1200 6396 50  0000 L CNN
+F 1 "MountingHole" H 1200 6305 50  0000 L CNN
+F 2 "Keyboard_Parts:MountingHole_M2" H 1100 6350 50  0001 C CNN
+F 3 "~" H 1100 6350 50  0001 C CNN
+	1    1100 6350
 	1    0    0    -1
 $EndComp
@@
 L Mechanical:MountingHole H2
 U 1 1 5F630832
-P 1700 4500
-F 0 "H2" H 1800 4546 50  0000 L CNN
-F 1 "MountingHole" H 1800 4455 50  0000 L CNN
-F 2 "Keyboard_Parts:MountingHole_M2" H 1700 4500 50  0001 C CNN
-F 3 "~" H 1700 4500 50  0001 C CNN
-	1    1700 4500
+P 1100 5950
+F 0 "H2" H 1200 5996 50  0000 L CNN
+F 1 "MountingHole" H 1200 5905 50  0000 L CNN
+F 2 "Keyboard_Parts:MountingHole_M2" H 1100 5950 50  0001 C CNN
+F 3 "~" H 1100 5950 50  0001 C CNN
+	1    1100 5950
 	1    0    0    -1
 $EndComp
@@
 L Mechanical:MountingHole H3
 U 1 1 5F630BA4
-P 1700 4700
-F 0 "H3" H 1800 4746 50  0000 L CNN
-F 1 "MountingHole" H 1800 4655 50  0000 L CNN
-F 2 "Keyboard_Parts:MountingHole_M2" H 1700 4700 50  0001 C CNN
-F 3 "~" H 1700 4700 50  0001 C CNN
-	1    1700 4700
-	1    0    0    -1
-$EndComp
+P 1100 6150
+F 0 "H3" H 1200 6196 50  0000 L CNN
+F 1 "MountingHole" H 1200 6105 50  0000 L CNN
+F 2 "Keyboard_Parts:MountingHole_M2" H 1100 6150 50  0001 C CNN
+F 3 "~" H 1100 6150 50  0001 C CNN
+	1    1100 6150
+	1    0    0    -1
+$EndComp
